Commit message: robot_update

File: projects/vision_controller/robot/ffw.urdf (robot description, URDF)
Before this commit: robot ffw, 35 links, 34 joints
Links:
- added link left_elbow_tcp
- added link left_hand_tcp
- added link right_elbow_tcp
- added link right_hand_tcp
Joints:
- added joint left_elbow_tcp_joint: type fixed, parent arm_l_link3, child left_elbow_tcp, origin xyz=0.04 0.0 -0.13 rpy=0 0 0
- added joint left_hand_tcp_joint: type fixed, parent arm_l_link7, child left_hand_tcp, origin xyz=0 0 0 rpy=0 0 0
- added joint right_elbow_tcp_joint: type fixed, parent arm_r_link3, child right_elbow_tcp, origin xyz=0.04 0.0 -0.13 rpy=0 0 0
- added joint right_hand_tcp_joint: type fixed, parent arm_r_link7, child right_hand_tcp, origin xyz=0.0 0.0 0.0 rpy=0 0 0
- joint world_to_base_yaw_joint: limit (none) -> lower=-3.14 upper=3.14 effort=100 velocity=1.0; type continuous -> revolute

Commit message: right arm add

File: projects/vision_controller/robot/ffw.urdf (robot description, URDF)
Before this commit: robot ffw, 39 links, 38 joints
Joints:
- joint left_hand_tcp_joint: origin xyz=0 0 0 rpy=0 0 0 -> xyz=0 0 -0.06 rpy=0 0 0
- joint right_hand_tcp_joint: origin xyz=0.0 0.0 0.0 rpy=0 0 0 -> xyz=0.0 0.0 -0.06 rpy=0 0 0
